File: v0_1/ChargerIC.kicad_sch (KiCad schematic)
At the start: 1 part, among them IC1 TP4056-42-ESOP8

Commit message: slide switch
Parts:
- added S1: MK-12C02-G020, MK-12C02-G020:MK12C02G020, symbol MK-12C02-G020:MK-12C02-G020
Changed lines of the file:
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@@
+    )
+  )
+  (symbol (lib_id "MK-12C02-G020:MK-12C02-G020") (at 106.68 62.23 0) (unit 1)
+    (in_bom yes) (on_board yes) (dnp no) (fields_autoplaced)
+    (property "Reference" "S1" (at 119.38 54.61 0)
+      (effects (font (size 1.27 1.27)))
+    )
+    (property "Value" "MK-12C02-G020" (at 119.38 57.15 0)
+      (effects (font (size 1.27 1.27)))
+    )
+    (property "Footprint" "MK-12C02-G020:MK12C02G020" (at 128.27 59.69 0)
+      (effects (font (size 1.27 1.27)) (justify left) hide)
+    )
+    (property "Datasheet" "https://datasheet.lcsc.com/lcsc/2012062037_G-Switch-MK-12C02-G020_C963206.pdf" (at 128.27 62.23 0)
+      (effects (font (size 1.27 1.27)) (justify left) hide)
+    )
+    (property "Description" "Surface Mount 1A SPDT 4.7mm 6V 6.6mm Black 2.7mm SMDSplicing 10000 Rectangular columnar -20~{+70} SMD Slide Switches ROHS" (at 128.27 64.77 0)
+      (effects (font (size 1.27 1.27)) (justify left) hide)
+    )
+    (property "Height" "1.45" (at 128.27 67.31 0)
+      (effects (font (size 1.27 1.27)) (justify left) hide)
+    )
+    (property "Manufacturer_Name" "G-Switch Electronic" (at 128.27 69.85 0)
+      (effects (font (size 1.27 1.27)) (justify left) hide)
+    )
+    (property "Manufacturer_Part_Number" "MK-12C02-G020" (at 128.27 72.39 0)
+      (effects (font (size 1.27 1.27)) (justify left) hide)
+    )
+    (property "Mouser Part Number" "" (at 128.27 74.93 0)
+      (effects (font (size 1.27 1.27)) (justify left) hide)
+    )
+    (property "Mouser Price/Stock" "" (at 128.27 77.47 0)
+      (effects (font (size 1.27 1.27)) (justify left) hide)
+    )
+    (property "Arrow Part Number" "" (at 128.27 80.01 0)
+      (effects (font (size 1.27 1.27)) (justify left) hide)
+    )
+    (property "Arrow Price/Stock" "" (at 128.27 82.55 0)
+      (effects (font (size 1.27 1.27)) (justify left) hide)
+    )
+    (pin "1")
+    (pin "2")
+    (pin "3")
+    (pin "MP1")
+    (pin "MP2")
+    (pin "MP3")
+    (pin "MP4")
+    (instances
+      (project "v0_1"
+        (path "/0bf090f4-b9b7-437f-9e6a-e818f47752ec/c0e4d80e-0821-408a-b2fe-ad88b3705532"
+          (reference "S1") (unit 1)
+        )
+      )
     )
   )

Commit message: charger ic circuit
Parts:
- added BT1: Battery, symbol Device:Battery
- added C1, C2: 10uF, symbol Device:C
- added D1: G-LED, symbol Device:LED
- added D2: R-LED, symbol Device:LED
- added R1: 0.4, symbol Device:R
- added R2: R-Prog, symbol Device:R
- added R3, R4: 1K, symbol Device:R
- added R5, R6: R, symbol Device:R
- added TH1: Thermistor_NTC, symbol Device:Thermistor_NTC
Connections:
- net at IC1.1 (TEMP): now also R5.2, R6.1, TH1.2
- net at IC1.2 (PROG): now also R2.1
- net at IC1.4 (VCC): now also IC1.8 (CE), C1.1, D1.2 (A), D2.2 (A), R1.2, R5.1
- net at IC1.5 (BAT): now also BT1.1 (+), C2.1
- net at IC1.6 (~{STDBY}): now also R3.2
- net at IC1.7 (~{CHRG}): now also R4.2
- new net: BT1.2 (-), TH1.1
- new net: D1.1 (K), R3.1
- new net: D2.1 (K), R4.1
- new net GND: C1.2, C2.2, R2.2, R6.2
- new net VCC: R1.1
Other:
- moved on the sheet: IC1, S1
