File: v0_1/Mico-USB-Charger.kicad_sch (KiCad schematic)
At the start: 14 parts, among them IC2 MCP73831T-2ACI_OT, J4 MICROQTJ, J5 S2B-PH-SM4-TB_LF__SN_

Commit message: add 0.2V
Connections:
- net 5V: now reaches C4.1, D3.2 (A), IC2.4 (VDD), J4.1, TP1.2
Changed lines of the file:
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@@
   (junction (at 196.85 86.36) (diameter 0) (color 0 0 0 0)
   )
+  (junction (at 119.38 74.93) (diameter 0) (color 0 0 0 0)
+  )
   (junction (at 156.21 111.76) (diameter 0) (color 0 0 0 0)
   )
@@
     (stroke (width 0) (type default))
   )
+  (wire (pts (xy 119.38 68.58) (xy 119.38 74.93))
+    (stroke (width 0) (type default))
+  )
   (wire (pts (xy 156.21 111.76) (xy 156.21 113.03))
     (stroke (width 0) (type default))
@@
     (stroke (width 0) (type default))
   )
+  (wire (pts (xy 119.38 68.58) (xy 120.65 68.58))
+    (stroke (width 0) (type default))
+  )
   (wire (pts (xy 208.28 88.9) (xy 208.28 111.76))
     (stroke (width 0) (type default))
@@
     (stroke (width 0) (type default))
   )
+  (wire (pts (xy 119.38 74.93) (xy 165.1 74.93))
+    (stroke (width 0) (type default))
+  )
   (wire (pts (xy 217.17 88.9) (xy 208.28 88.9))
     (stroke (width 0) (type default))
@@
     (stroke (width 0) (type default))
   )
+  (wire (pts (xy 105.41 74.93) (xy 119.38 74.93))
+    (stroke (width 0) (type default))
+  )
   (wire (pts (xy 133.35 88.9) (xy 133.35 111.76))
     (stroke (width 0) (type default))
@@
     (stroke (width 0) (type default))
   )
-  (wire (pts (xy 105.41 74.93) (xy 165.1 74.93))
-    (stroke (width 0) (type default))
-  )
   (wire (pts (xy 115.57 83.82) (xy 119.38 83.82))
     (stroke (width 0) (type default))
@@
     (stroke (width 0) (type default))
   )
+  (hierarchical_label "5V" (shape input) (at 120.65 68.58 0) (fields_autoplaced)
+    (effects (font (size 1.27 1.27)) (justify left))
+  )
   (symbol (lib_id "Device:R") (at 123.19 83.82 90) (unit 1)
