File: v0_1/v0_1.kicad_pcb (KiCad board)
At the start: 2 copper layers, 4 parts, among them J1 Z-ICS0S40P-W000, U1 Pico, U2 PCF8523T, U3 AHT20

Commit message: add charger ic
Parts:
- added IC1: TP4056-42-ESOP8, TP4056:SOIC127P600X175-9N, F.Cu at (53.2, 92.1)
Changed lines of the file:
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@@
   (net 96 "unconnected-(U3-GND-Pad5)")
   (net 97 "unconnected-(U3-NC_2-Pad6)")
+  (net 98 "unconnected-(IC1-TEMP-Pad1)")
+  (net 99 "unconnected-(IC1-PROG-Pad2)")
+  (net 100 "unconnected-(IC1-GND-Pad3)")
+  (net 101 "unconnected-(IC1-VCC-Pad4)")
+  (net 102 "unconnected-(IC1-BAT-Pad5)")
+  (net 103 "unconnected-(IC1-~{STDBY}-Pad6)")
+  (net 104 "unconnected-(IC1-~{CHRG}-Pad7)")
+  (net 105 "unconnected-(IC1-CE-Pad8)")
+  (net 106 "unconnected-(IC1-EP-Pad9)")
   (footprint "Z-ICS0S40P-W000:ZICS0S40PW000" (layer "F.Cu")
     (at 88.9 111.76 90)
@@
     (property "Mouser Part Number" "")
     (property "Mouser Price/Stock" "")
-    (property "Sheetfile" "Picowhttpsensor.kicad_sch")
+    (property "Sheetfile" "v0_1.kicad_sch")
     (property "Sheetname" "")
     (property "ki_description" "DIP Tin 15.24mm 40 2.54mm DIP-40  IC Sockets ROHS")
@@
     (descr "Through hole straight pin header, 2x20, 2.54mm pitch, double rows")
     (tags "Through hole pin header THT 2x20 2.54mm double row")
-    (property "Sheetfile" "Picowhttpsensor.kicad_sch")
+    (property "Sheetfile" "v0_1.kicad_sch")
     (property "Sheetname" "")
     (attr through_hole)
@@
       (net 43 "unconnected-(U1-SWDIO-Pad43)") (pinfunction "SWDIO") (pintype "bidirectional"))
   )
+  (footprint "TP4056:SOIC127P600X175-9N" (layer "F.Cu")
+    (at 53.168 92.075)
+    (descr "8ESOP")
+    (tags "Integrated Circuit")
+    (property "Arrow Part Number" "")
+    (property "Arrow Price/Stock" "")
+    (property "Description" "PMIC - Battery Management ESOP-8 RoHS")
+    (property "Height" "1.75")
+    (property "Manufacturer_Name" "Nanjing Extension Microelectronics")
+    (property "Manufacturer_Part_Number" "TP4056-42-ESOP8")
+    (property "Mouser Part Number" "")
+    (property "Mouser Price/Stock" "")
+    (property "Sheetfile" "v0_1.kicad_sch")
+    (property "Sheetname" "")
+    (property "ki_description" "PMIC - Battery Management ESOP-8 RoHS")
+    (attr smd)
+    (fp_text reference "IC1" (at 0 0) (layer "F.SilkS")
+        (effects (font (size 1.27 1.27) (thickness 0.254)))
+    )
+    (fp_text value "TP4056-42-ESOP8" (at 0 0) (layer "F.SilkS") hide
+        (effects (font (size 1.27 1.27) (thickness 0.254)))
+    )
+    (fp_text user "${REFERENCE}" (at 0 0) (layer "F.Fab")
+        (effects (font (size 1.27 1.27) (thickness 0.254)))
+    )
+    (fp_line (start -3.475 -2.605) (end -1.95 -2.605)
+      (stroke (width 0.2) (type solid)) (layer "F.SilkS"))
+    (fp_line (start -3.725 -2.8) (end 3.725 -2.8)
+      (stroke (width 0.05) (type solid)) (layer "F.CrtYd"))
+    (fp_line (start -3.725 2.8) (end -3.725 -2.8)
+      (stroke (width 0.05) (type solid)) (layer "F.CrtYd"))
+    (fp_line (start 3.725 -2.8) (end 3.725 2.8)
+      (stroke (width 0.05) (type solid)) (layer "F.CrtYd"))
+    (fp_line (start 3.725 2.8) (end -3.725 2.8)
+      (stroke (width 0.05) (type solid)) (layer "F.CrtYd"))
+    (fp_line (start -1.95 -2.45) (end 1.95 -2.45)
+      (stroke (width 0.1) (type solid)) (layer "F.Fab"))
+    (fp_line (start -1.95 -1.18) (end -0.68 -2.45)
+      (stroke (width 0.1) (type solid)) (layer "F.Fab"))
+    (fp_line (start -1.95 2.45) (end -1.95 -2.45)
+      (stroke (width 0.1) (type solid)) (layer "F.Fab"))
+    (fp_line (start 1.95 -2.45) (end 1.95 2.45)
+      (stroke (width 0.1) (type solid)) (layer "F.Fab"))
+    (fp_line (start 1.95 2.45) (end -1.95 2.45)
+      (stroke (width 0.1) (type solid)) (layer "F.Fab"))
+    (pad "1" smd rect (at -2.712 -1.905 90) (size 0.7 1.525) (layers "F.Cu" "F.Paste" "F.Mask")
+      (net 98 "unconnected-(IC1-TEMP-Pad1)") (pinfunction "TEMP") (pintype "passive"))
+    (pad "2" smd rect (at -2.712 -0.635 90) (size 0.7 1.525) (layers "F.Cu" "F.Paste" "F.Mask")
+      (net 99 "unconnected-(IC1-PROG-Pad2)") (pinfunction "PROG") (pintype "passive"))
+    (pad "3" smd rect (at -2.712 0.635 90) (size 0.7 1.525) (layers "F.Cu" "F.Paste" "F.Mask")
+      (net 100 "unconnected-(IC1-GND-Pad3)") (pinfunction "GND") (pintype "passive"))
+    (pad "4" smd rect (at -2.712 1.905 90) (size 0.7 1.525) (layers "F.Cu" "F.Paste" "F.Mask")
+      (net 101 "unconnected-(IC1-VCC-Pad4)") (pinfunction "VCC") (pintype "passive"))
+    (pad "5" smd rect (at 2.712 1.905 90) (size 0.7 1.525) (layers "F.Cu" "F.Paste" "F.Mask")
+      (net 102 "unconnected-(IC1-BAT-Pad5)") (pinfunction "BAT") (pintype "passive"))
+    (pad "6" smd rect (at 2.712 0.635 90) (size 0.7 1.525) (layers "F.Cu" "F.Paste" "F.Mask")
+      (net 103 "unconnected-(IC1-~{STDBY}-Pad6)") (pinfunction "~{STDBY}") (pintype "passive"))
+    (pad "7" smd rect (at 2.712 -0.635 90) (size 0.7 1.525) (layers "F.Cu" "F.Paste" "F.Mask")
+      (net 104 "unconnected-(IC1-~{CHRG}-Pad7)") (pinfunction "~{CHRG}") (pintype "passive"))
+    (pad "8" smd rect (at 2.712 -1.905 90) (size 0.7 1.525) (layers "F.Cu" "F.Paste" "F.Mask")
+      (net 105 "unconnected-(IC1-CE-Pad8)") (pinfunction "CE") (pintype "passive"))
+    (pad "9" smd rect (at 0 0) (size 2.513 3.402) (layers "F.Cu" "F.Paste" "F.Mask")
+      (net 106 "unconnected-(IC1-EP-Pad9)") (pinfunction "EP") (pintype "passive"))
+    (model "TP4056-42-ESOP8.stp"
+      (offset (xyz 0 0 0))
+      (scale (xyz 1 1 1))
+      (rotate (xyz 0 0 0))
+    )
+  )
   (footprint "AHT20:AHT20" (layer "F.Cu")
     (at 65.04 54.88)
@@
     (property "Mouser Part Number" "")
     (property "Mouser Price/Stock" "")
-    (property "Sheetfile" "Picowhttpsensor.kicad_sch")
+    (property "Sheetfile" "v0_1.kicad_sch")
     (property "Sheetname" "")
     (property "ki_description" "Integrated temperature and humidity Sensor DC : 2.2 - 5.5V, 0 ~ 100% RH, -40 ~ + 85 .")
@@
     (descr "SOIC, 8 Pin (JEDEC MS-012AA, https://www.analog.com/media/en/package-pcb-resources/package/pkg_pdf/soic_narrow-r/r_8.pdf), generated with kicad-footprint-generator ipc_gullwing_generator.py")
     (tags "SOIC SO")
-    (property "Sheetfile" "Picowhttpsensor.kicad_sch")
+    (property "Sheetfile" "v0_1.kicad_sch")
     (property "Sheetname" "")
     (property "ki_description" "Realtime Clock/Calendar I2C Interface, SOIC-8")

Commit message: save
Parts:
- added J2: HYCW110-TF10-180B, HYCW110-TF10-180B:HYCW110TF10180B, F.Cu at (119.9, 59.4)
- added J3: BS-12-B3AA009, BS-12-B3AA009:BS12B3AA009, F.Cu at (152.4, 58.4)
- added S1: MK-12C02-G020, MK-12C02-G020:MK12C02G020, F.Cu at (108.0, 100.5)
- moved IC1 57.1 mm to (107.8, 108.6)
- moved U2 57.1 mm to (110.6, 85.7)
- moved U1 57.1 mm to (172.7, 101.6)
- moved U3 57.1 mm to (119.7, 71.4)
- moved J1 57.1 mm to (143.5, 128.3)

Commit message: add rtc and charger schematic
Parts:
- added IC2: MCP73831T-2ACI_OT, MCP73831T_2ACIOT:SOT95P270X145-5N, F.Cu at (97.8, 67.6)
- added J4: MICROQTJ, MicroQTJ:MICROQTJ, F.Cu at (121.2, 38.5)
- added J5: S2B-PH-SM4-TB_LF__SN_, S2B-PH-SM4-TB(LF)(SN):S2BPHSM4TBLFSN, F.Cu at (98.1, 50.1)
- added Y1: MC-306_32.7680K-A0_ROHS, MC-306_32.7680K-A0ROHS:MC306327680KA5ROHS, F.Cu at (101.4, 84.8)
Connections:
- IC1 pad 1: unconnected-(IC1-TEMP-Pad1) -> Net-(IC1-TEMP)
- IC1 pad 2: unconnected-(IC1-PROG-Pad2) -> Net-(IC1-PROG)
- IC1 pad 4: unconnected-(IC1-VCC-Pad4) -> Net-(D1-A)
- IC1 pad 5: unconnected-(IC1-BAT-Pad5) -> Net-(BT1-+)
- IC1 pad 6: unconnected-(IC1-~{STDBY}-Pad6) -> Net-(IC1-~{STDBY})
- IC1 pad 7: unconnected-(IC1-~{CHRG}-Pad7) -> Net-(IC1-~{CHRG})
- IC1 pad 8: unconnected-(IC1-CE-Pad8) -> Net-(D1-A)

Commit message: add 0.2V
Parts:
- moved U2 10.2 mm to (119.4, 80.6)
Connections:
- IC2 pad 4: Net-(D3-A) -> +3.3V
- J2 pad 2: unconnected-(J2-CD/DAT_3-Pad2) -> /PCF8523T/SD_CS
- J2 pad 3: unconnected-(J2-CMD-Pad3) -> /PCF8523T/MOSI
- J2 pad 4: unconnected-(J2-VDD-Pad4) -> VCC
- J2 pad 5: unconnected-(J2-CLK-Pad5) -> /PCF8523T/SCK
- J2 pad 6: unconnected-(J2-VSS-Pad6) -> GND
- J2 pad 7: unconnected-(J2-DAT0-Pad7) -> /PCF8523T/MISO
- J2 pad G1: unconnected-(J2-GROUND_1-PadG1) -> GND
- J2 pad G2: unconnected-(J2-GROUND_2-PadG2) -> GND
- J3 pad 1: unconnected-(J3---Pad1) -> GND
- J3 pad 2: unconnected-(J3-+-Pad2) -> Net-(J3-+)
- J4 pad 1: Net-(D3-A) -> +3.3V
- U1 pad 13: unconnected-(U1-GND-Pad13) -> GND
- U1 pad 18: unconnected-(U1-GND-Pad18) -> GND
- U1 pad 21: unconnected-(U1-GPIO16-Pad21) -> /MISO
- U1 pad 22: unconnected-(U1-GPIO17-Pad22) -> /SD_CS
- U1 pad 23: unconnected-(U1-GND-Pad23) -> GND
- U1 pad 24: unconnected-(U1-GPIO18-Pad24) -> /SCK
- U1 pad 25: unconnected-(U1-GPIO19-Pad25) -> /MOSI
- U1 pad 28: unconnected-(U1-GND-Pad28) -> GND
- U1 pad 3: unconnected-(U1-GND-Pad3) -> GND
- U1 pad 36: unconnected-(U1-3V3-Pad36) -> +3.3V
- U1 pad 38: unconnected-(U1-GND-Pad38) -> GND
- U1 pad 6: unconnected-(U1-GPIO4-Pad6) -> /SCL
- U1 pad 7: unconnected-(U1-GPIO5-Pad7) -> /SDA
- U1 pad 8: unconnected-(U1-GND-Pad8) -> GND
- U2 pad 1: unconnected-(U2-OSCI-Pad1) -> Net-(U2-OSCI)
- U2 pad 2: unconnected-(U2-OSCO-Pad2) -> Net-(U2-OSCO)
- U2 pad 3: unconnected-(U2-VBAT-Pad3) -> Net-(J3-+)
- U2 pad 4: unconnected-(U2-VSS-Pad4) -> GND
- U2 pad 5: unconnected-(U2-SDA-Pad5) -> /PCF8523T/SDA
- U2 pad 6: unconnected-(U2-SCL-Pad6) -> /PCF8523T/SCL
- U2 pad 7: unconnected-(U2-~{INT1}/CLKOUT-Pad7) -> Net-(J6-Pin_1)
- U2 pad 8: unconnected-(U2-VDD-Pad8) -> Net-(U2-VDD)
- U3 pad 2: unconnected-(U3-VDD-Pad2) -> VCC
- Y1 pad 1: unconnected-(Y1-CRYSTAL_1-Pad1) -> Net-(U2-OSCO)
- Y1 pad 4: unconnected-(Y1-CRYSTAL_2-Pad4) -> Net-(U2-OSCI)
