File: v0_2/HYCW110TF10180B.kicad_sch (KiCad schematic)
At the start: 4 parts, among them J2 HYCW110-TF10-180B, J3 Conn_01x09_Pin

Commit message: rename i2c and add button
Parts:
- J2: footprint HYCW110TF10180B -> HYCW110-TF10-180B:HYCW110TF10180B
Connections:
- net CARDDET: now also J2.10 (COM), R3.2
Changed lines of the file:
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@@
     (effects (font (size 1.27 1.27)) (justify left bottom))
   )
-  (label "CARDDET" (at 168.91 107.95 0) (fields_autoplaced)
-    (effects (font (size 1.27 1.27)) (justify left bottom))
+  (label "CARDDET" (at 195.58 105.41 180) (fields_autoplaced)
+    (effects (font (size 1.27 1.27)) (justify right bottom))
   )
   (label "CARDDET" (at 73.66 107.95 0) (fields_autoplaced)
@@
       (effects (font (size 1.27 1.27)))
     )
-    (property "Footprint" "HYCW110TF10180B" (at 156.21 82.55 0)
+    (property "Footprint" "HYCW110-TF10-180B:HYCW110TF10180B" (at 156.21 82.55 0)
       (effects (font (size 1.27 1.27)) (justify left) hide)
     )

Commit message: power line
Parts:
- removed J3: Conn_01x09_Pin, Connector_PinHeader_1.27mm:PinHeader_1x09_P1.27mm_Vertical, symbol Connector:Conn_01x09_Pin
- added TP5, TP6, TP7, TP8: TestPoint, TestPoint:TestPoint_Pad_D1.0mm, symbol Connector:TestPoint
Connections:
- net CS: now also TP6.1
- net DIN: now also TP5.1
- net DO: now also TP8.1
- net SCLK: now also TP7.1
