File: v0_2/v0_2.kicad_sch (KiCad schematic)
At the start: 21 parts, among them IC1 RASPBERRY_PI_PICO_W

Commit message: power line
Parts:
- added TP10, TP11, TP9: TestPoint, TestPoint:TestPoint_Pad_D1.0mm, symbol Connector:TestPoint
Connections:
- net +3.3V: now also TP9.1
- net GND: now also IC1.33 (GND/AGND), TP10.1
- net V+_A0: now also TP11.1
- net DQ: now reaches IC1.34 (GP28/ADC2)
Other:
- added sheet TemperatureOutdoor (DS18B20.kicad_sch)
- moved on the sheet: D3A, D3B, R15
