File: v0_2_5/AHT20.kicad_sch (KiCad schematic)
At the start: 3 parts, among them U1 AHT20

Commit message: replace sdcard
Parts:
- U1: LCSC (none) -> C3012622
Changed lines of the file:
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@@
       (effects (font (size 1.27 1.27)) (justify left) hide)
+    )
+    (property "LCSC" "C3012622" (at 124.46 91.44 0)
+      (effects (font (size 1.27 1.27)) hide)
     )
     (pin "1")
