File: v0_2_5/BH1750FVI.kicad_sch (KiCad schematic)
At the start: 5 parts, among them IC2 BH1750FVI-TR

Commit message: replace sdcard
Parts:
- JP1: now left out of the parts list
Changed lines of the file:
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@@
   )
   (symbol (lib_id "Jumper:SolderJumper_2_Open") (at 104.14 92.71 0) (unit 1)
-    (in_bom yes) (on_board yes) (dnp no) (fields_autoplaced)
+    (in_bom no) (on_board no) (dnp no) (fields_autoplaced)
     (property "Reference" "JP1" (at 104.14 86.36 0)
       (effects (font (size 1.27 1.27)))
