File: v0_2_5/SM04B-SRSS-TB.kicad_sch (KiCad schematic)
At the start: 1 part, among them J4 SM04B-SRSS-TB

Commit message: replace sdcard
Parts:
- J4: LCSC (none) -> C160404
Changed lines of the file:
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@@
       (effects (font (size 1.27 1.27)) (justify left) hide)
+    )
+    (property "LCSC" "C160404" (at 104.14 72.39 0)
+      (effects (font (size 1.27 1.27)) hide)
     )
     (pin "1")
