File: v0_2_5/AP2138N-3.3TRG1.kicad_sch (KiCad schematic)
At the start: 10 parts, among them IC3 AP2138N-3.3TRG1, J1 S2B-PH-SM4-TB_LF__SN_, J6 Conn_01x02_Pin, Q1 DMG2301L-7, Q2 DMG2301L-7, Q5 DMN3731U-7

Commit message: replace sdcard
Parts:
- J1: LCSC (none) -> S2B-PH-SM4-TB
- J6: now left out of the parts list
Changed lines of the file:
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@@
       (effects (font (size 1.27 1.27)) (justify left) hide)
+    )
+    (property "LCSC" "S2B-PH-SM4-TB" (at 243.84 87.63 0)
+      (effects (font (size 1.27 1.27)) hide)
     )
     (pin "1")
@@
   )
   (symbol (lib_id "Connector:Conn_01x02_Pin") (at 238.76 96.52 0) (unit 1)
-    (in_bom yes) (on_board yes) (dnp no) (fields_autoplaced)
+    (in_bom no) (on_board no) (dnp no) (fields_autoplaced)
     (property "Reference" "J6" (at 239.395 91.44 0)
       (effects (font (size 1.27 1.27)))
