File: v0_2_5/DS18B20.kicad_sch (KiCad schematic)
At the start: 4 parts, among them J5 Screw_Terminal_01x03, U3 DS18B20

Commit message: replacement
Parts:
- removed U3: DS18B20, Package_TO_SOT_THT:TO-92_Inline, symbol Sensor_Temperature:DS18B20
Changed lines of the file:
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@@
 (kicad_sch (version 20230121) (generator eeschema)
   (paper "A4")
-  (junction (at 111.76 58.42) (diameter 0) (color 0 0 0 0)
-  )
-  (junction (at 130.81 58.42) (diameter 0) (color 0 0 0 0)
-  )
   (junction (at 134.62 83.82) (diameter 0) (color 0 0 0 0)
   )
   (junction (at 121.92 83.82) (diameter 0) (color 0 0 0 0)
   )
-  (junction (at 121.92 72.39) (diameter 0) (color 0 0 0 0)
-  )
   (junction (at 130.81 72.39) (diameter 0) (color 0 0 0 0)
-  )
-  (wire (pts (xy 134.62 58.42) (xy 130.81 58.42))
-    (stroke (width 0) (type default))
   )
   (wire (pts (xy 121.92 72.39) (xy 121.92 83.82))
@@
   )
   (wire (pts (xy 134.62 83.82) (xy 138.43 83.82))
-    (stroke (width 0) (type default))
-  )
-  (wire (pts (xy 114.3 58.42) (xy 111.76 58.42))
     (stroke (width 0) (type default))
   )
@@
     (stroke (width 0) (type default))
   )
-  (wire (pts (xy 129.54 58.42) (xy 130.81 58.42))
-    (stroke (width 0) (type default))
-  )
-  (wire (pts (xy 121.92 66.04) (xy 121.92 72.39))
-    (stroke (width 0) (type default))
-  )
   (wire (pts (xy 107.95 58.42) (xy 111.76 58.42))
     (stroke (width 0) (type default))
   )
-  (wire (pts (xy 130.81 58.42) (xy 130.81 72.39))
+  (wire (pts (xy 130.81 57.15) (xy 130.81 72.39))
     (stroke (width 0) (type default))
   )
@@
   )
   (wire (pts (xy 121.92 83.82) (xy 134.62 83.82))
-    (stroke (width 0) (type default))
-  )
-  (wire (pts (xy 134.62 57.15) (xy 134.62 58.42))
     (stroke (width 0) (type default))
   )
@@
     (pin "2")
     (instances
-      (project "v0_2"
+      (project "v0_2_5"
         (path "/678523e5-508b-4706-b0e0-f17e466a8d09"
           (reference "R13") (unit 1)
@@
     )
   )
-  (symbol (lib_id "power:+3.3V") (at 134.62 57.15 0) (unit 1)
+  (symbol (lib_id "power:+3.3V") (at 130.81 57.15 0) (unit 1)
     (in_bom yes) (on_board yes) (dnp no) (fields_autoplaced)
-    (property "Reference" "#PWR035" (at 134.62 60.96 0)
+    (property "Reference" "#PWR035" (at 130.81 60.96 0)
       (effects (font (size 1.27 1.27)) hide)
     )
-    (property "Value" "+3.3V" (at 134.62 52.07 0)
+    (property "Value" "+3.3V" (at 130.81 52.07 0)
       (effects (font (size 1.27 1.27)))
     )
-    (property "Footprint" "" (at 134.62 57.15 0)
+    (property "Footprint" "" (at 130.81 57.15 0)
       (effects (font (size 1.27 1.27)) hide)
     )
-    (property "Datasheet" "" (at 134.62 57.15 0)
+    (property "Datasheet" "" (at 130.81 57.15 0)
       (effects (font (size 1.27 1.27)) hide)
     )
     (pin "1")
     (instances
-      (project "v0_2"
+      (project "v0_2_5"
         (path "/678523e5-508b-4706-b0e0-f17e466a8d09/21f03d30-0ecc-439b-8de2-493752139474"
           (reference "#PWR035") (unit 1)
@@
     (pin "1")
     (instances
-      (project "v0_2"
+      (project "v0_2_5"
         (path "/678523e5-508b-4706-b0e0-f17e466a8d09/21f03d30-0ecc-439b-8de2-493752139474"
           (reference "#PWR034") (unit 1)
@@
     (pin "3")
     (instances
-      (project "v0_2"
+      (project "v0_2_5"
         (path "/678523e5-508b-4706-b0e0-f17e466a8d09/21f03d30-0ecc-439b-8de2-493752139474"
           (reference "J5") (unit 1)
-        )
-      )
-    )
-  )
-  (symbol (lib_id "Sensor_Temperature:DS18B20") (at 121.92 58.42 270) (unit 1)
-    (in_bom yes) (on_board yes) (dnp no) (fields_autoplaced)
-    (property "Reference" "U3" (at 121.92 48.26 90)
-      (effects (font (size 1.27 1.27)))
-    )
-    (property "Value" "DS18B20" (at 121.92 50.8 90)
-      (effects (font (size 1.27 1.27)))
-    )
-    (property "Footprint" "Package_TO_SOT_THT:TO-92_Inline" (at 115.57 33.02 0)
-      (effects (font (size 1.27 1.27)) hide)
-    )
-    (property "Datasheet" "http://datasheets.maximintegrated.com/en/ds/DS18B20.pdf" (at 128.27 54.61 0)
-      (effects (font (size 1.27 1.27)) hide)
-    )
-    (pin "1")
-    (pin "2")
-    (pin "3")
-    (instances
-      (project "v0_2"
-        (path "/678523e5-508b-4706-b0e0-f17e466a8d09/21f03d30-0ecc-439b-8de2-493752139474"
-          (reference "U3") (unit 1)
         )
       )
@@
     (pin "1")
     (instances
-      (project "v0_2"
+      (project "v0_2_5"
         (path "/678523e5-508b-4706-b0e0-f17e466a8d09"
           (reference "TP11") (unit 1)

Commit message: change for manufacture
Parts:
- J5: LCSC (none) -> C5188441
Changed lines of the file:
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@@
+      (effects (font (size 1.27 1.27)) hide)
+    )
+    (property "LCSC" "C5188441" (at 102.87 83.82 0)
       (effects (font (size 1.27 1.27)) hide)
     )

Commit message: replace sdcard
Parts:
- J5: LCSC C5188441 -> (none); LCSC Part # (none) -> C5188441; now left out of the parts list
- TP11: now left out of the parts list
Changed lines of the file:
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@@
   )
   (symbol (lib_id "Connector:Screw_Terminal_01x03") (at 102.87 83.82 180) (unit 1)
-    (in_bom yes) (on_board yes) (dnp no) (fields_autoplaced)
+    (in_bom no) (on_board no) (dnp no) (fields_autoplaced)
     (property "Reference" "J5" (at 102.87 74.93 0)
       (effects (font (size 1.27 1.27)))
@@
       (effects (font (size 1.27 1.27)) hide)
     )
-    (property "LCSC" "C5188441" (at 102.87 83.82 0)
+    (property "LCSC Part #" "C5188441" (at 102.87 83.82 0)
       (effects (font (size 1.27 1.27)) hide)
     )
@@
   )
   (symbol (lib_id "Connector:TestPoint") (at 134.62 83.82 0) (unit 1)
-    (in_bom yes) (on_board yes) (dnp no) (fields_autoplaced)
+    (in_bom no) (on_board no) (dnp no) (fields_autoplaced)
     (property "Reference" "TP11" (at 137.16 79.248 0)
       (effects (font (size 1.27 1.27)) (justify left))
