File: v0_2_5/v0_2_5.kicad_sch (KiCad schematic)
At the start: 24 parts, among them IC1 RASPBERRY_PI_PICO_W

Commit message: replacement
Connections:
- net GND: now also IC1.13 (GND_3), IC1.18 (GND_4), IC1.23 (GND_5), IC1.28 (GND_6), IC1.3 (GND_1), IC1.38 (GND_7), IC1.8 (GND_2)

Commit message: change placement
Connections:
- net Record: now also IC1.17 (UART0_RX/I2C0_SCL_/SPI1_CSN/GP13); no longer IC1.16 (UART0_TX/I2C0_SDA_/SPI1_RX_/GP12)
Other:
- moved on the sheet: TP10
Changed lines of the file:
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@@
+    (stroke (width 0) (type default))
+  )
+  (wire (pts (xy 26.67 74.93) (xy 50.8 74.93))
     (stroke (width 0) (type default))
   )
@@
   )
   (wire (pts (xy 163.83 36.83) (xy 163.83 29.21))
-    (stroke (width 0) (type default))
-  )
-  (wire (pts (xy 26.67 72.39) (xy 50.8 72.39))
     (stroke (width 0) (type default))
   )
@@
     (effects (font (size 1.27 1.27)) (justify left bottom))
   )
-  (label "Record" (at 26.67 72.39 0) (fields_autoplaced)
-    (effects (font (size 1.27 1.27)) (justify left bottom))
-  )
   (label "ACT_LED" (at 26.67 54.61 0) (fields_autoplaced)
     (effects (font (size 1.27 1.27)) (justify left bottom))
@@
     (effects (font (size 1.27 1.27)) (justify left bottom))
   )
+  (label "Record" (at 26.67 74.93 0) (fields_autoplaced)
+    (effects (font (size 1.27 1.27)) (justify left bottom))
+  )
   (label "I2C0_SDA" (at 91.44 128.27 0) (fields_autoplaced)
     (effects (font (size 1.27 1.27)) (justify left bottom))
@@
     (effects (font (size 1.27 1.27)) (justify left bottom))
   )
-  (symbol (lib_id "Connector:TestPoint") (at 173.99 52.07 270) (unit 1)
-    (in_bom yes) (on_board yes) (dnp no) (fields_autoplaced)
-    (property "Reference" "TP10" (at 179.07 50.8 90)
+  (symbol (lib_id "Connector:TestPoint") (at 173.99 52.07 90) (mirror x) (unit 1)
+    (in_bom yes) (on_board yes) (dnp no)
+    (property "Reference" "TP10" (at 168.91 50.8 90)
       (effects (font (size 1.27 1.27)) (justify left))
     )
-    (property "Value" "TestPoint" (at 179.07 53.34 90)
+    (property "Value" "TestPoint" (at 168.91 53.34 90)
       (effects (font (size 1.27 1.27)) (justify left))
     )

Commit message: replace sdcard
Parts:
- TP1, TP2, TP3, TP4: now left out of the parts list
Changed lines of the file:
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@@
   )
   (symbol (lib_id "Connector:TestPoint") (at 78.74 137.16 0) (unit 1)
-    (in_bom yes) (on_board yes) (dnp no) (fields_autoplaced)
+    (in_bom no) (on_board no) (dnp no) (fields_autoplaced)
     (property "Reference" "TP3" (at 81.28 132.588 0)
       (effects (font (size 1.27 1.27)) (justify left))
@@
   )
   (symbol (lib_id "Connector:TestPoint") (at 78.74 128.27 0) (unit 1)
-    (in_bom yes) (on_board yes) (dnp no) (fields_autoplaced)
+    (in_bom no) (on_board no) (dnp no) (fields_autoplaced)
     (property "Reference" "TP2" (at 81.28 123.698 0)
       (effects (font (size 1.27 1.27)) (justify left))
@@
   )
   (symbol (lib_id "Connector:TestPoint") (at 78.74 146.05 0) (unit 1)
-    (in_bom yes) (on_board yes) (dnp no) (fields_autoplaced)
+    (in_bom no) (on_board no) (dnp no) (fields_autoplaced)
     (property "Reference" "TP4" (at 81.28 141.478 0)
       (effects (font (size 1.27 1.27)) (justify left))
@@
   )
   (symbol (lib_id "Connector:TestPoint") (at 78.74 119.38 0) (unit 1)
-    (in_bom yes) (on_board yes) (dnp no) (fields_autoplaced)
+    (in_bom no) (on_board no) (dnp no) (fields_autoplaced)
     (property "Reference" "TP1" (at 81.28 114.808 0)
       (effects (font (size 1.27 1.27)) (justify left))

Commit message: replace sdcard
Parts:
- TP11: now left out of the parts list
Changed lines of the file:
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@@
   )
   (symbol (lib_id "Connector:TestPoint") (at 78.74 137.16 0) (unit 1)
-    (in_bom no) (on_board no) (dnp no) (fields_autoplaced)
+    (in_bom no) (on_board yes) (dnp no) (fields_autoplaced)
     (property "Reference" "TP3" (at 81.28 132.588 0)
       (effects (font (size 1.27 1.27)) (justify left))
@@
   )
   (symbol (lib_id "Connector:TestPoint") (at 78.74 128.27 0) (unit 1)
-    (in_bom no) (on_board no) (dnp no) (fields_autoplaced)
+    (in_bom no) (on_board yes) (dnp no) (fields_autoplaced)
     (property "Reference" "TP2" (at 81.28 123.698 0)
       (effects (font (size 1.27 1.27)) (justify left))
@@
   )
   (symbol (lib_id "Connector:TestPoint") (at 78.74 146.05 0) (unit 1)
-    (in_bom no) (on_board no) (dnp no) (fields_autoplaced)
+    (in_bom no) (on_board yes) (dnp no) (fields_autoplaced)
     (property "Reference" "TP4" (at 81.28 141.478 0)
       (effects (font (size 1.27 1.27)) (justify left))
@@
   )
   (symbol (lib_id "Connector:TestPoint") (at 271.78 73.66 270) (unit 1)
-    (in_bom yes) (on_board yes) (dnp no) (fields_autoplaced)
+    (in_bom no) (on_board yes) (dnp no) (fields_autoplaced)
     (property "Reference" "TP11" (at 276.86 72.39 90)
       (effects (font (size 1.27 1.27)) (justify left))
@@
   )
   (symbol (lib_id "Connector:TestPoint") (at 78.74 119.38 0) (unit 1)
-    (in_bom no) (on_board no) (dnp no) (fields_autoplaced)
+    (in_bom no) (on_board yes) (dnp no) (fields_autoplaced)
     (property "Reference" "TP1" (at 81.28 114.808 0)
       (effects (font (size 1.27 1.27)) (justify left))
